Commit message: test assets

File: nimble/bottle.urdf (robot description, URDF)
Before this commit: robot bottle_skeleton, 2 links, 1 joints
Joints:
- joint bot: origin xyz=0.4 0 0.4 rpy=-1.57075 0 0 -> xyz=0.4 0.3 0.4 rpy=1.5 0 0

File: nimble/ground.urdf (robot description, URDF)
Before this commit: robot ground_skeleton, 2 links, 1 joints
Links:
- link ground_link: geometry collision box size=2.0 0.3 2.0; visual box size=2.0 0.3 2.0

Commit message: bottle to box

File: nimble/bottle.urdf (robot description, URDF)
Before this commit: robot bottle_skeleton, 2 links, 1 joints
Links:
- link bottle_free: geometry collision box size=0.05 0.05 0.2; visual box size=0.05 0.05 0.2
Joints:
- joint bot: origin xyz=0.4 0.3 0.4 rpy=1.5 0 0 -> xyz=-0.5 0.2 0.05 rpy=-1.57075 0 0
