Commit message: urdf change

File: nimble/ur5_gripper_no_col.urdf (robot description, URDF)
Before this commit: robot ur5, 14 links, 13 joints
Links:
- link base_link: geometry visual mesh filename=meshes/ur5/visual/base.stl
- link ee_link: geometry visual box size=0.01 0.01 0.01
- link forearm_link: geometry visual mesh filename=meshes/ur5/visual/forearm.stl
- link left_inner_finger: geometry collision mesh filename=box.obj scale=0.005 0.01 0.02; visual mesh filename=box.obj scale=0.005 0.01 0.02
- link left_inner_knuckle: geometry visual mesh filename=meshes/ur5/visual/inner_knuckle_coarse.stl
- link right_inner_finger: geometry collision mesh filename=box.obj scale=0.005 0.01 0.02; visual mesh filename=box.obj scale=0.005 0.01 0.02
- link right_inner_knuckle: geometry visual mesh filename=meshes/ur5/visual/inner_knuckle_coarse.stl
- link robotiq_base_link: geometry visual mesh filename=meshes/ur5/visual/robotiq_85_base_link_coarse.stl
- link shoulder_link: geometry visual mesh filename=meshes/ur5/visual/shoulder.stl
- link upper_arm_link: geometry visual mesh filename=meshes/ur5/visual/upperarm.stl
- link wrist_1_link: geometry visual mesh filename=meshes/ur5/visual/wrist1.stl
- link wrist_2_link: geometry visual mesh filename=meshes/ur5/visual/wrist2.stl
- link wrist_3_link: geometry visual mesh filename=meshes/ur5/visual/wrist3.stl
Joints:
- joint base_to_lik: limit lower=-1 upper=1 effort=20 velocity=3.2 -> lower=-0.3 upper=0.8 effort=20 velocity=3.2
- joint base_to_rik: limit lower=-1 upper=1 effort=20 velocity=3.2 -> lower=-0.3 upper=0.8 effort=20 velocity=3.2
