Commit message: nimble assets

File: nimble/box1.urdf (robot description, URDF)
Before this commit: robot bottle_skeleton, 2 links, 1 joints
Links:
- link bottle_free: mass 1.0 -> 0.0001; geometry collision mesh filename=box.obj scale=0.02 0.08 0.02; visual mesh filename=box.obj scale=0.02 0.08 0.02
Joints:
- joint bot: origin xyz=-0.5 0.2 0.05 rpy=-1.57075 0 0 -> xyz=-0.5 0.07 0.035 rpy=0 0 0
