Commit message: assets update

File: nimble/ground_obj.urdf (robot description, URDF)
Before this commit: robot ground_skeleton, 2 links, 1 joints
Joints:
- joint ground_joint: origin xyz=0 -.2 0 rpy=0 0 0 -> xyz=0 -.06 0 rpy=0 0 0

File: nimble/ur5_gripper_ee_bottle.urdf (robot description, URDF)
Before this commit: robot ur5, 15 links, 14 joints
Links:
- added link bottle_link, mass 1.0; visual mesh filename=new_bottle/bottle.obj scale=0.001 0.0023 0.001
Joints:
- added joint bottle_fixed: type fixed, parent robotiq_base_link, child bottle_link, origin xyz=0 0.05 0.16 rpy=0 0 3.1415
