Commit message: Add revolute joint

File: nimble/new_bottle/bottle_and_cap.urdf (robot description, URDF)
Before this commit: robot bottle_and_cap.urdf, 2 links, 1 joints
Joints:
- joint cap_joint: type fixed -> revolute

Commit message: scaling

File: nimble/new_bottle/bottle_and_cap.urdf (robot description, URDF)
Before this commit: robot bottle_and_cap.urdf, 2 links, 1 joints
Links:
- added link world
- link bottle: mass None -> 0.0001; geometry collision mesh filename=bottle.obj scale=.002 .002 .002; visual mesh filename=bottle.obj scale=.002 .002 .002
- link cap: mass None -> 0.0001; geometry collision mesh filename=cap.obj scale=.002 .002 .002; visual mesh filename=cap.obj scale=.002 .002 .002
Joints:
- added joint bot: type floating, parent world, child bottle, origin xyz=-0.5 0.1 0.035 rpy=0 0 0
- joint cap_joint: origin xyz=0 .6 0 rpy=0 0 0 -> xyz=0 .12 0 rpy=0 0 0; type revolute -> fixed
